File: small_laser_supply_eagleproj/small_laser_supply/small_laser_supply.sch (EAGLE design)
At the start: 0 parts

Commit message: Added a board with the general parts layout, and a general layout of the schematic as well.
Parts:
- added MH1, MH2, MH3, MH4: THREADED_INSERT_M3, small_laser_supply_lib:THREADED_INSERT_M3
- added X1: 5V_IN, small_laser_supply_lib:BNC_TE-VERT-PTH
- added X2: CTRL, small_laser_supply_lib:BNC_TE-VERT-PTH
- added X3: OUT, small_laser_supply_lib:BNC_TE-VERT-PTH
Connections:
- new net GND: MH1.P, MH2.P, MH3.P, MH4.P, X1.GND, X2.GND, X3.GND
